File: ebus-adapter.kicad_sch (KiCad schematic)
At the start: 0 parts

Commit message: Updated adapter added SPI 2 Etherenet adapter
Parts:
- added C1: 100n, Capacitor_SMD:C_0603_1608Metric_Pad1.08x0.95mm_HandSolder, symbol Device:C
- added C10, C4, C6: 100u, Capacitor_SMD:C_0603_1608Metric_Pad1.08x0.95mm_HandSolder, symbol Device:C
- added C11, C18, C2, C3, C7: 10u, Capacitor_SMD:C_0603_1608Metric_Pad1.08x0.95mm_HandSolder, symbol Device:C
- added C12, C5, C8: 100p, Capacitor_SMD:C_0603_1608Metric_Pad1.08x0.95mm_HandSolder, symbol Device:C
- added C13, C14: 18p, Capacitor_SMD:C_0603_1608Metric_Pad1.08x0.95mm_HandSolder, symbol Device:C
- added C15, C16, C17, C22: 10n, Capacitor_SMD:C_0603_1608Metric_Pad1.08x0.95mm_HandSolder, symbol Device:C
- added C19: 22n, Capacitor_SMD:C_0603_1608Metric_Pad1.08x0.95mm_HandSolder, symbol Device:C
- added C20, C21: 6.8n, Capacitor_SMD:C_0603_1608Metric_Pad1.08x0.95mm_HandSolder, symbol Device:C
- added C23: 1n/2kV, Capacitor_SMD:C_0603_1608Metric_Pad1.08x0.95mm_HandSolder, symbol Device:C
- added C24, C25: C, Capacitor_SMD:C_0603_1608Metric_Pad1.08x0.95mm_HandSolder, symbol Device:C
- added C9: 4.7u, Capacitor_SMD:C_0603_1608Metric_Pad1.08x0.95mm_HandSolder, symbol Device:C
- added D1, D2: BAV99, Package_TO_SOT_SMD:SOT-23, symbol Diode:BAV99
- added D3: LED, symbol Device:LED
- added D4: 7.5V/1W, Diode_SMD:D_SOD-123, symbol Device:D_Zener
- added D5: 24V/1W, Diode_SMD:D_SOD-123, symbol Device:D_Zener
- added D6: 3.9V, Diode_SMD:D_SOD-123, symbol Device:D_Zener
- added FB1: 120 Ohm @ 100 MHz, symbol Device:FerriteBead_Small
- added J1, J2: Conn_01x02_Socket, Connector_Molex:Molex_PicoBlade_53047-0210_1x02_P1.25mm_Vertical, symbol Connector:Conn_01x02_Socket
- added J3: HR911105A, ebus-adapter-footprints:HR911105A, symbol ebus-adapter-library:HR911105A
- added J4: WJ2EDGRC-5.08-2P, ebus-adapter-footprints:WJ2EDGRC, symbol Connector:Conn_01x02_Socket
- added J5: PWR, ebus-adapter-footprints:WJ2EDGRC, symbol Connector:Conn_Coaxial_Power
- added Q1, Q2: BC817, Package_TO_SOT_SMD:SOT-23, symbol Transistor_BJT:BC817
- added Q3: DMN13H750S, Package_TO_SOT_SMD:SOT-23, symbol Transistor_FET:DMN13H750S
- added R1, R6: 100k, Resistor_SMD:R_0603_1608Metric_Pad0.98x0.95mm_HandSolder, symbol Device:R
- added R10, R12, R20, R7: 10k, Resistor_SMD:R_0603_1608Metric_Pad0.98x0.95mm_HandSolder, symbol Device:R
- added R11: 0, Resistor_SMD:R_0603_1608Metric_Pad0.98x0.95mm_HandSolder, symbol Device:R
- added R13: 12.4k 1%, Resistor_SMD:R_0603_1608Metric_Pad0.98x0.95mm_HandSolder, symbol Device:R
- added R14: 1M, Resistor_SMD:R_0603_1608Metric_Pad0.98x0.95mm_HandSolder, symbol Device:R
- added R15, R16, R18, R19: 49.9 1%, Resistor_SMD:R_0603_1608Metric_Pad0.98x0.95mm_HandSolder, symbol Device:R
- added R17: 10 1%, Resistor_SMD:R_0603_1608Metric_Pad0.98x0.95mm_HandSolder, symbol Device:R
- added R2: 33k, Resistor_SMD:R_0603_1608Metric_Pad0.98x0.95mm_HandSolder, symbol Device:R
- added R3: R, Resistor_SMD:R_0603_1608Metric_Pad0.98x0.95mm_HandSolder, symbol Device:R
- added R4: 4k7, Resistor_SMD:R_0603_1608Metric_Pad0.98x0.95mm_HandSolder, symbol Device:R
- added R5: 2M, Resistor_SMD:R_0603_1608Metric_Pad0.98x0.95mm_HandSolder, symbol Device:R
- added R8, R9: 330, Resistor_SMD:R_0603_1608Metric_Pad0.98x0.95mm_HandSolder, symbol Device:R
- added SW1: SW_Push_Dual, symbol Switch:SW_Push_Dual
- added TP1: EBUS_RX, TestPoint:TestPoint_Loop_D1.80mm_Drill1.0mm_Beaded, symbol Connector:TestPoint
- added TP2: EBUS_SIG, TestPoint:TestPoint_Loop_D1.80mm_Drill1.0mm_Beaded, symbol Connector:TestPoint
- added TP3: EBUS_RX_LL, TestPoint:TestPoint_Loop_D1.80mm_Drill1.0mm_Beaded, symbol Connector:TestPoint
- added TP4: EBUS_3.3, TestPoint:TestPoint_Loop_D1.80mm_Drill1.0mm_Beaded, symbol Connector:TestPoint
- added TP5: BOOT0, TestPoint:TestPoint_Loop_D1.80mm_Drill1.0mm_Beaded, symbol Connector:TestPoint
- added TP6: GND1, TestPoint:TestPoint_Loop_D1.80mm_Drill1.0mm_Beaded, symbol Connector:TestPoint
- added TP7: GND2, TestPoint:TestPoint_Loop_D1.80mm_Drill1.0mm_Beaded, symbol Connector:TestPoint
- added TP8: 3.3V, TestPoint:TestPoint_Loop_D1.80mm_Drill1.0mm_Beaded, symbol Connector:TestPoint
- added U1: LM358DR, Package_SO:SOIC-8_3.9x4.9mm_P1.27mm, symbol Device:Opamp_Dual
- added U2: ADuM1201BR, Package_SO:SOIC-8_3.9x4.9mm_P1.27mm, symbol Isolator:ADuM1201BR
- added U3: STM32L412KBTx, Package_QFP:LQFP-32_7x7mm_P0.8mm, symbol MCU_ST_STM32L4:STM32L412KBTx
- added U4: W5500, Package_QFP:LQFP-48_7x7mm_P0.5mm, symbol Interface_Ethernet:W5500
- added U5: W25Q128JVSIQ, Package_SO:SOIC-8_5.23x5.23mm_P1.27mm, symbol Memory_Flash:W25Q32JVSS
- added U6: AMS1117-3.3, Package_TO_SOT_SMD:SOT-223-3_TabPin2, symbol Regulator_Linear:AMS1117-3.3
- added Y1: YSX321SL @24Mhz, ebus-adapter-footprints:YSX321SL, symbol ebus-adapter-library:YSX321SL
Connections:
- new net: C13.1, R14.1, U4.30 (XI/CLKIN), Y1.1
- new net: C14.1, R14.2, U4.31 (XO), Y1.3
- new net: R1.2, R2.1, R5.1, TP1.1, U1.5 (+)
- new net: C9.1, U4.20 (TOCAP)
- new net: Q1.1 (B), R4.2
- new net: D4.2 (A), Q1.3 (C)
- new net: D3.2 (A), R3.2
- new net: J5.1 (In), Q3.3 (D)
- new net: R4.1, U1.1
- new net: C23.1, J3.8 (GND)
- new net: C15.1, U4.22 (1V2O)
- new net: D1.3 (K), J4.2 (Pin_2)
- new net: R12.2, U4.43 (PMODE2), U4.44 (PMODE1), U4.45 (PMODE0)
- new net: C1.1, D6.1 (K), Q2.1 (B), R6.2
- new net: C22.1, J3.5 (RCT), R18.2, R19.2
- new net: R13.1, U4.10 (EXRES1)
- new net: C24.1, Q3.2 (S), U6.3 (VI)
- new net: J3.9 (GLED-), R8.2
- new net: R11.2, U3.26 (PB3)
- new net: D2.3 (K), J4.1 (Pin_1)
- new net: C19.1, J3.4 (TCT), R17.2
- new net: C20.2, J3.3 (RXD+)
- new net: J3.12 (YLED-), R9.1
- new net: C21.2, J3.6 (RXD-)
- new net +3.3V: C10.1, C11.1, C12.1, C16.1, C25.1, C3.1, C4.1, C5.1, C6.1, C7.1, C8.1, FB1.1, R10.1, R12.1, R7.1, R8.1, R9.2, TP8.1, U2.8 (VDD2), U3.1 (VDD), U3.17 (VDD), U3.5 (VDDA), U6.2 (VO)
- new net +3.3VA: C17.1, C18.1, FB1.2, R15.1, R16.1, R17.1, U4.11 (AVDD), U4.15 (AVDD), U4.17 (AVDD), U4.21 (AVDD), U4.4 (AVDD), U4.8 (AVDD)
- new net BOOT0: R20.1, TP5.1, U3.31 (PH3)
- new net EBUS_3.3V: C2.1, J1.1 (Pin_1), Q2.2 (E), TP4.1, U1.2 (-), U1.6 (-), U1.8 (V+), U2.1 (VDD1)
- new net EBUS_SIGNAL: D1.2 (A), D2.2 (A), D4.1 (K), D5.1 (K), Q2.3 (C), R1.1, R6.1, TP2.1
- new net ETHER_CS: U3.29 (PB6), U4.32 (~{SCS})
- new net ETHER_INT: U3.28 (PB5), U4.36 (~{INT})
- new net GND1: C1.2, C2.2, D1.1 (K), D2.1 (K), D5.2 (A), D6.2 (A), J1.2 (Pin_2), Q1.2 (E), R2.2, TP6.1, U1.4 (V-), U2.4 (GND1)
- new net GND2: C10.2, C11.2, C12.2, C13.2, C14.2, C15.2, C16.2, C17.2, C18.2, C19.2, C22.2, C23.2, C24.2, C25.2, C3.2, C4.2, C5.2, C6.2, C7.2, C8.2, C9.2, J5.2 (Ext), Q3.1 (G), R13.2, R20.2, SW1.1, SW1.3, TP7.1, U2.5 (GND2), U3.16 (VSS), U3.32 (VSS), U4.14 (AGND), U4.16 (AGND), U4.19 (AGND), U4.23 (RSVD), U4.28 (VDD), U4.29 (GND), U4.3 (AGND), U4.38 (RSVD), U4.39 (RSVD), U4.40 (RSVD), U4.41 (RSVD), U4.42 (RSVD), U4.48 (AGND), U4.9 (AGND), U5.4 (GND), U5.8 (VCC), U6.1 (GND), Y1.2, Y1.4
- new net LNK_LED: J3.10 (GLED+), U4.25 (LINKLED)
- new net NRST: R7.2, SW1.2, U3.4 (NRST)
- new net NRST_MCU: R10.2, SW1.4, U3.27 (PB4), U4.37 (~{RST})
- new net QUADSPI_BK1_IO0: U3.15 (PB1), U5.5 (DI(IO0))
- new net QUADSPI_BK1_IO1: U3.14 (PB0), U5.2 (DO(IO1))
- new net QUADSPI_BK1_IO2: U3.13 (PA7), U5.3 (IO2)
- new net QUADSPI_BK1_IO3: U3.12 (PA6), U5.7 (IO3)
- new net QUADSPI_BK1_NCS: U3.8 (PA2), U5.1 (~{CS})
- new net QUADSPI_CLK: U3.9 (PA3), U5.6 (CLK)
- new net RX: U2.6 (VOB), U3.20 (PA10)
- new net RX+: C20.1, R18.1, U4.6 (RXP)
- new net RX-: C21.1, R19.1, U4.5 (RXN)
- new net SPD_LED: J3.11 (YLED+), U4.24 (SPDLED)
- new net SPI_MISO: U3.21 (PA11), U4.34 (MISO)
- new net SPI_MOSI: U3.22 (PA12), U4.35 (MOSI)
- new net SPI_SCK: U3.7 (PA1), U4.33 (SCLK)
- new net SWCLK: U3.24 (PA14)
- new net SWDIO: U3.23 (PA13)
- new net SWO: R11.1
- new net TX: U2.7 (VIA), U3.19 (PA9)
- new net TX+: J3.1 (TXD+), R16.2, U4.2 (TXP)
- new net TX-: J3.2 (TXD-), R15.2, U4.1 (TXN)
- new net VIB: R5.2, TP3.1, U1.7, U2.3 (VIB)
- new net VOA: U1.3 (+), U2.2 (VOA)
- new net _EBUS_PWR: J2.2 (Pin_2), R3.1
- new net _GND1: D3.1 (K), J2.1 (Pin_1)
- no-connect marks 0 -> 4
Other:
- removed sheet Ebus-To-UART
- note added: "22-6V"
- note added: "24-8V"
- note added: "6-2.2V"

Commit message: Updated schematics and pcb
Parts:
- removed C14: 18p, Capacitor_SMD:C_0603_1608Metric_Pad1.08x0.95mm_HandSolder, symbol Device:C
- removed C15, C22: 10n, Capacitor_SMD:C_0603_1608Metric_Pad1.08x0.95mm_HandSolder, symbol Device:C
- removed C19: 22n, Capacitor_SMD:C_0603_1608Metric_Pad1.08x0.95mm_HandSolder, symbol Device:C
- removed C20, C21: 6.8n, Capacitor_SMD:C_0603_1608Metric_Pad1.08x0.95mm_HandSolder, symbol Device:C
- removed R19: 49.9 1%, Resistor_SMD:R_0603_1608Metric_Pad0.98x0.95mm_HandSolder, symbol Device:R
- removed SW1: SW_Push_Dual, symbol Switch:SW_Push_Dual
- removed U4: W5500, Package_QFP:LQFP-48_7x7mm_P0.5mm, symbol Interface_Ethernet:W5500
- added D7: LED, LED_THT:LED_D1.8mm_W3.3mm_H2.4mm, symbol Device:LED
- added FB2: 120 Ohm @ 100 MHz, Resistor_SMD:R_1206_3216Metric_Pad1.30x1.75mm_HandSolder, symbol Device:FerriteBead
- added J6: Conn_01x05_Pin, Connector_PinHeader_2.54mm:PinHeader_1x05_P2.54mm_Vertical, symbol Connector:Conn_01x05_Pin
- added J7, J8: Conn_01x02_Socket, Connector_Molex:Molex_PicoBlade_53047-0210_1x02_P1.25mm_Vertical, symbol Connector:Conn_01x02_Socket
- added SW2: PS-7054SVB-6PN, ebus-adapter-footprints:PS-7054SVB, symbol Switch:SW_Push_DPDT
- added U4: ENC28J60x-ML, Package_DFN_QFN:QFN-28-1EP_6x6mm_P0.65mm_EP4.25x4.25mm, symbol Interface_Ethernet:ENC28J60x-ML
- C6: value 100u -> 10uF
- C7: value 10u -> 0.1uF
- C8: value 100p -> 0.1uF
- C9: value 4.7u -> 18p
- D3: footprint (none) -> LED_THT:LED_D1.8mm_W3.3mm_H2.4mm
- FB1: footprint (none) -> Resistor_SMD:R_1206_3216Metric_Pad1.30x1.75mm_HandSolder; Part Name (none) -> YI321611Z121-6R0T; Part Number (none) -> C3011219
- J3: Part Name (none) -> HR911105A
- J4, J5: Part Name (none) -> WJ2EDGRC-5.08-2P
- R12: value 10k -> 2.32k 1%
- R13: value 12.4k 1% -> 49.9 1%
- R14: value 1M -> 49.9 1%
- R17: value 10 1% -> 1M
- R18: value 49.9 1% -> R
- TP1, TP2, TP3, TP4, TP5, TP6, TP7, TP8: footprint TestPoint:TestPoint_Loop_D1.80mm_Drill1.0mm_Beaded -> TestPoint:TestPoint_THTPad_1.5x1.5mm_Drill0.7mm
- Y1: value YSX321SL @24Mhz -> YSX321SL @25Mhz
Connections:
- net +3.3V: now also U5.8 (VCC), J6.2 (Pin_2); no longer C6.1, C7.1, C8.1, R12.1
- net +3.3VA: now also FB2.1, U4.11 (VDDTX), U4.15 (VDDRX), U4.16 (VDDPLL), U4.21 (VDDOSC), U4.24 (VDD); no longer R15.1, R16.1, R17.1
- net EBUS_3.3V: now also R3.1; no longer J1.1 (Pin_1)
- net ETHER_CS: now also U4.5 (~{CS})
- net ETHER_INT: now also U4.28 (~{INT})
- net GND2: now also C7.1, C8.1, R12.2, J6.1 (Pin_1), J7.2 (Pin_2), SW2.2 (B), SW2.5 (B), U4.14 (VSSTX), U4.17 (VSSPLL), U4.18 (VSSOSC), U4.26 (VSS), U4.7 (VSSRX); no longer C7.2, C8.2, R13.2, U5.8 (VCC)
- net LNK_LED: now also U4.23 (LEDA)
- net NRST: now also SW2.3 (C)
- net NRST_MCU: now also SW2.6 (C), U4.6 (~{RESET})
- net RX+: now also J3.3 (RXD+), R13.2, U4.13 (TPOUT+); no longer R18.1
- net RX-: now also J3.6 (RXD-), R14.2, U4.12 (TPOUT-)
- net SPD_LED: now also U4.22 (LEDB)
- net SWCLK: now also J6.4 (Pin_4)
- net SWDIO: now also J6.3 (Pin_3)
- net SWO: now also J6.5 (Pin_5)
- net TX+: now also R15.2, U4.9 (TPIN+); no longer R16.2
- net TX-: now also R16.2, U4.8 (TPIN-); no longer R15.2
- net _EBUS_PWR: now also D3.2 (A); no longer R3.1
- net at Y1.3: now also C13.1, R17.1; no longer R14.2
- net at C9.1: now also Y1.1, U4.19 (OSC1)
- net at R3.2: now also J1.1 (Pin_1); no longer D3.2 (A)
- net at J3.5 (RCT): now also C8.2, R13.1, R14.1; no longer R18.2
- net at R17.2: now also U4.20 (OSC2); no longer J3.4 (TCT)
- net ACT: now reaches U3.10 (PA4)
- net ACT: now also R18.1
- net SPI_MISO renamed ETHER_DI
- net ETHER_DI: now also U4.2 (SO)
- net SPI_MOSI renamed ETHER_DO
- net ETHER_DO: now also U4.3 (SI)
- net SPI_SCK renamed ETHER_SCK
- net ETHER_SCK: now also U4.4 (SCK)
- new net: C6.1, U4.25 (VCAP)
- new net: J7.1 (Pin_1), R18.2
- new net: C7.2, FB2.2, J3.4 (TCT), R15.1, R16.1
- new net: R12.1, U4.10 (RBIAS)
- new net _ACT: D7.2 (A), J8.2 (Pin_2)
- new net _GND2: D7.1 (K), J8.1 (Pin_1)
- no-connect marks 4 -> 12
Other:
- moved on the sheet: C10, C11, C12, C23, J3, R10, R15, R16, R8, R9, U5
